Commit message: Updated parameters

File: urdf/udacity_bot.xacro (robot description, xacro)
@@ -37,5 +37,5 @@
       <origin xyz="-0.15 0 -0.05" rpy=" 0 0 0"/>
       <geometry>
-        <sphere radius="0.05"/>
+        <sphere radius="0.0495"/>
       </geometry>
       <surface>
@@ -59,5 +59,5 @@
       <origin xyz="0.15 0 -0.05" rpy=" 0 0 0"/>
       <geometry>
-        <sphere radius="0.05"/>
+        <sphere radius="0.0495"/>
       </geometry>
       <surface>
